Commit message: Se implementa el robot en rviz hasta el tercer link

File: laboratorio_4_robotica/urdf/4r_robot_gazebo.xacro (robot description, xacro)
@@ -18,12 +18,12 @@
      izz="0.01"
      />
-     <xacro:m_joint name="${joint_01_name}"
+     <xacro:m_joint name="joint_1"
      type="revolute"
      axis_xyz="0 0 1"
-     origin_rpy="0 0 0" origin_xyz="0 0 0.094375"
-     parent="${link_00_name}" child="${link_01_name}"
+     origin_rpy="0 0 -1.5708" origin_xyz="0 0 0.094375"
+     parent="${link_00_name}" child="link_1"
      limit_e="10" limit_l="-3.14" limit_u="3.14" limit_v="5.0"
      />
-     <xacro:m_link_mesh name="${link_01_name}"
+     <xacro:m_link_mesh name="link_1"
      origin_xyz="0 0 0.0"
      origin_rpy="0 0 0"
@@ -34,3 +34,35 @@
      izz="0.01"
      />
+     <xacro:m_joint name="joint_2"
+     type="revolute"
+     axis_xyz="0 0 1"
+     origin_rpy="1.5708 -1.5708 1.5708" origin_xyz="0 0 0.0415"
+     parent="link_1" child="link_2"
+     limit_e="10" limit_l="-3.14" limit_u="3.14" limit_v="5.0"
+     />
+     <xacro:m_link_mesh name="link_2"
+     origin_xyz="-0.011 0 0"
+     origin_rpy="0 0 0"
+     meshfile="package://laboratorio_4_robotica/meshes/PincherLink2.stl"
+     mass="1"
+     ixx="0.01" ixy="0" ixz="0"
+     iyy="0.01" iyz="0"
+     izz="0.01"
+     />
+     <xacro:m_joint name="joint_3"
+     type="revolute"
+     axis_xyz="0 0 1"
+     origin_rpy="0 0 0" origin_xyz="0.107 0 0"
+     parent="link_2" child="link_3"
+     limit_e="10" limit_l="-3.14" limit_u="3.14" limit_v="5.0"
+     />
+     <xacro:m_link_mesh name="link_3"
+     origin_xyz="-0.0115 0 0"
+     origin_rpy="0 0 0"
+     meshfile="package://laboratorio_4_robotica/meshes/PincherLink3.stl"
+     mass="0.5"
+     ixx="0.01" ixy="0" ixz="0"
+     iyy="0.01" iyz="0"
+     izz="0.01"
+     />
 </robot>

File: laboratorio_4_robotica/urdf/robot_parameters.xacro (robot description, xacro)
@@ -2,11 +2,11 @@
 <robot xmlns:xacro="http://www.ros.org/wiki/xacro">
   <xacro:property name="link_00_name" value="robot_base" />
-  <xacro:property name="link_01_name" value="link_01" />
-  <xacro:property name="link_02_name" value="link_02" />
-  <xacro:property name="link_03_name" value="finger_1" />
+  <xacro:property name="link_01_name" value="link_1" />
+  <xacro:property name="link_02_name" value="link_2" />
+  <xacro:property name="link_03_name" value="link_3" />
   <xacro:property name="link_04_name" value="finger_2" />
   <xacro:property name="joint_01_name" value="joint_1" />
   <xacro:property name="joint_02_name" value="joint_2" />
-  <xacro:property name="joint_03_name" value="gripper_1" />
+  <xacro:property name="joint_03_name" value="joint_3" />
   <xacro:property name="joint_04_name" value="gripper_2" />
 </robot>

Commit message: Se arreglan problemas de referencia y se cambia el material dentro de gazebo.

File: laboratorio_4_robotica/urdf/4r_robot_gazebo.xacro (robot description, xacro)
@@ -1,6 +1,6 @@
 <?xml version="1.0"?>
 <robot xmlns:xacro="http://www.ros.org/wiki/xacro" name="4R_robot">
-     <xacro:include filename="$(find basic_2r_gazebo)/urdf/links_joints.xacro" />
-     <xacro:include filename="$(find basic_2r_gazebo)/urdf/robot_parameters.xacro" />
+     <xacro:include filename="$(find laboratorio_4_robotica)/urdf/links_joints.xacro" />
+     <xacro:include filename="$(find laboratorio_4_robotica)/urdf/robot_parameters.xacro" />
      <xacro:include filename="$(find laboratorio_4_robotica)/urdf/my_macros.xacro"/>
      <link name="world"/>  <!-- Base link from Gazebo-->

File: laboratorio_4_robotica/urdf/links_joints.xacro (robot description, xacro)
@@ -50,5 +50,5 @@
         <origin rpy="${origin_rpy}" xyz="${origin_xyz}" />
         <geometry>
-          <mesh filename="${meshfile}" scale="1.0 1.0 1.0"/>
+          <mesh filename="${meshfile}" scale="0.1 0.1 0.1"/>
         </geometry>
       </collision>
@@ -56,5 +56,5 @@
         <origin rpy="${origin_rpy}" xyz="${origin_xyz}" />
         <geometry>
-          <mesh filename="${meshfile}" scale="1.0 1.0 1.0"/>
+          <mesh filename="${meshfile}" scale="0.1 0.1 0.1"/>
         </geometry>
         <material name="Cyan">
@@ -64,5 +64,5 @@
     </link>
     <gazebo reference="${name}">
-        <material>Gazebo/BlueGlow</material>
+        <material>Gazebo/BlackTransparent</material>
     </gazebo>
  </xacro:macro>

File: laboratorio_4_robotica/urdf/robot_parameters.xacro (robot description, xacro)
@@ -2,11 +2,11 @@
 <robot xmlns:xacro="http://www.ros.org/wiki/xacro">
   <xacro:property name="link_00_name" value="robot_base" />
-  <xacro:property name="link_01_name" value="link_1" />
-  <xacro:property name="link_02_name" value="link_2" />
-  <xacro:property name="link_03_name" value="link_3" />
+  <xacro:property name="link_01_name" value="link_01" />
+  <xacro:property name="link_02_name" value="link_02" />
+  <xacro:property name="link_03_name" value="finger_1" />
   <xacro:property name="link_04_name" value="finger_2" />
   <xacro:property name="joint_01_name" value="joint_1" />
   <xacro:property name="joint_02_name" value="joint_2" />
-  <xacro:property name="joint_03_name" value="joint_3" />
+  <xacro:property name="joint_03_name" value="gripper_1" />
   <xacro:property name="joint_04_name" value="gripper_2" />
 </robot>

Commit message: Se desarrolla el modelo del robot en matlab y se valida el movimiento correcto de las articulaciones

File: laboratorio_4_robotica/urdf/4r_robot_gazebo.xacro (robot description, xacro)
@@ -4,6 +4,6 @@
      <xacro:include filename="$(find laboratorio_4_robotica)/urdf/robot_parameters.xacro" />
      <xacro:include filename="$(find laboratorio_4_robotica)/urdf/my_macros.xacro"/>
-     <link name="world"/>  <!-- Base link from Gazebo-->
-     <joint name="fixed" type="fixed"> <!-- Joint to fix the base so it does not move-->
+     <link name="world"/>
+     <joint name="fixed" type="fixed">
           <parent link="world"/>
           <child link="${link_00_name}"/>
@@ -115,5 +115,4 @@
      izz="0.00000178"
      />
-     <!--
      <xacro:create_noa name="NOA"
      origin_xyz="0.305 0 0"
@@ -121,6 +120,4 @@
      parent="link_2"
      />
-     -->
-     <!-- Gazebo Plugin -->
      <gazebo>
        <plugin name="gazebo_ros_control" filename="libgazebo_ros_control.so">
