Commit message: Se implementa el publicador que controla las articulaciones y el suscriptor que lee las posiciones desde Matlab

File: laboratorio_4_robotica/urdf/links_joints.xacro (robot description, xacro)
@@ -64,4 +64,5 @@
     </link>
     <gazebo reference="${name}">
+        <!--<material>Gazebo/WhiteGlow</material>-->
         <material>Gazebo/BlackTransparent</material>
     </gazebo>
